File: hardware/hmesh/rev_a/hmesh.sch (EAGLE design)
At the start: 26 parts, among them P1 MOLEX_73251-135X, P2 MOLEX_73251-135X, U1 ATUM, U2 CC110L, U3 AS3930-BQFT, X1 ABS05-32.768KHZ-9-T, X2 M416F26022CKR

Commit message: updated schematic
Parts:
- removed J12: (no value), SparkFun-Passives:JUMPER-2PTH
- added JP1, JP2: JUMPER-3PTH, SparkFun-Passives:JUMPER-3PTH
- added Q1, Q2: MOSFET-NCHANNELSMD, fets:MOSFET-NCHANNELSMD
Connections:
- removed net I2C_SDA: J12.1
- removed net I2C_SDA_FTDI: J12.2
- removed net N$26: D3.C
- new net CC110L_GDO0_SW: JP1.1
- new net CC110L_GDO2_SW: JP2.1
- new net N$13: D3.C, Q2.D
- new net N$14: JP1.3, Q1.G
- new net N$15: JP2.3, Q2.G
- net CC110L_GDO0: now also JP1.2
- net CC110L_GDO2: now also JP2.2
- net GND: now also Q1.S, Q2.S
- net N$12: now also Q1.D

Commit message: pretty good board made
Parts:
- added C12: 0.1uF, passives:CAPACITOR
- added H1, H2, H3, H4: MOUNT-HOLE3.2, holes:MOUNT-HOLE3.2
- added J1: TC2030-CC2538-BL, connector:TC2030-CC2538-BL
- added J2: TC2030-CTX, connector:TC2030-CTX
- added JP3: (no value), pinhead:PINHD-2X10
- added JP4, JP5, JP6: JUMPER-3PTH, SparkFun-Passives:JUMPER-3PTH
- added JP7: (no value), pinhead:PINHD-1X2
- JP1, JP2: value JUMPER-3PTH -> (none); device SparkFun-Passives:JUMPER-3PTH -> SparkFun-Passives:JUMPER-2PTH
Connections:
- removed net CC110L_GDO0_SW: JP1.1
- removed net CC110L_GDO2_SW: JP2.1
- removed net N$11: C10.1, C11.1, C6.1, C7.1, C8.1, C9.1, U2.AVDD, U2.DGUARD, U2.DVDD
- removed net N$5: R1.2, U3.VCC
- removed net VCC3V3: R3.2, R4.2
- new net AS3930_CS: JP3.3, JP3.4, U1.B5, U3.CS
- new net AS3930_DAT: JP3.5, JP3.6, U1.B4, U3.DAT
- new net AS3930_WAKE: JP3.7, JP3.8, U1.B3, U3.WAKE
- new net N$17: J1.TX, U1.BTLDR_TX
- new net N$18: J1.RX, U1.BTLDR_RX
- new net N$19: J1.BL_CTRL, U1.BTLDR_CTRL
- new net N$20: J1.!RESET, J2.!RESET, U1.!RESET
- new net N$22: J2.TMS, U1.TMS
- new net N$23: J2.TCK, U1.TCK
- new net N$26: J2.TDO, U1.TDO
- new net VCC: JP4.3, JP5.3, JP6.3, JP7.1, JP7.2, R3.2, R4.2
- new net VCC_AS3930: C12.1, JP4.1, JP4.2, R1.2, U3.VCC
- new net VCC_ATUM: J1.VCC, J2.VCC, JP6.1, JP6.2, U1.VCC
- new net VCC_CC110L: C10.1, C11.1, C6.1, C7.1, C8.1, C9.1, JP5.1, JP5.2, U2.AVDD, U2.DGUARD, U2.DVDD
- net !CC110L_CS: now also JP3.15, JP3.16, U1.C2
- net CC110L_GDO0: now also JP2.1, JP3.17, JP3.18, U1.C1; no longer JP1.2
- net CC110L_GDO2: now also JP1.1, JP3.19, JP3.20, U1.C0; no longer JP2.2
- net GND: now also C12.2, J1.GND, J2.GND, JP3.1, JP3.2, U1.GND, U3.GND
- net MISO: now also JP3.10, JP3.9, U1.SPI_MISO, U3.MISO
- net MOSI: now also JP3.11, JP3.12, U1.SPI_MOSI, U3.MOSI
- net N$14: now also JP2.2; no longer JP1.3
- net N$15: now also JP1.2; no longer JP2.3
- net SCLK: now also JP3.13, JP3.14, U1.SPI_SCK, U3.SCLK
Other:
- note added: "PIN 18"
- note added: "PIN 4"
